File: in14-4.sch (EAGLE design)
At the start: 15 parts, among them IC1 4094D, IC2 4094D, Q1 K155ID1, Q2 K155ID1, Q3 K155ID1, Q4 K155ID1

Commit message: .
Parts:
- removed IC2: 4094D, 40xx:4094D
- added IC3: 4094D, 40xx:4094D
Connections:
- net +5V: no longer JP1.3
- net N$24: now also IC3A.Q2; no longer IC1A.Q2
- net N$28: now also IC3A.Q6; no longer IC1A.Q6
- net N$29: now also IC3A.Q7; no longer IC1A.Q7
- net N$30: now also IC3A.Q8; no longer IC1A.Q8
- net N$31: now also IC3A.D; no longer IC1A.D
- net N$32: now also IC3A.CLK; no longer IC2A.CLK
- net N$33: now also IC3A.STR; no longer IC2A.STR
- net N$34: now also IC3A.OE; no longer IC2A.OE
- net N$35: now also IC1A.Q4; no longer IC2A.Q4
- net N$36: now also IC1A.Q3; no longer IC2A.Q3
- net N$37: now also IC1A.Q2; no longer IC2A.Q2
- net N$38: now also IC1A.Q1; no longer IC2A.Q1
- net N$39: now also IC1A.Q5; no longer IC2A.Q5
- net N$40: now also IC1A.Q6; no longer IC2A.Q6
- net N$41: now also IC1A.Q7; no longer IC2A.Q7
- net N$42: now also IC1A.Q8; no longer IC2A.Q8
- net N$63: now also IC3A.Q1; no longer IC1A.Q1
- net N$67: now also IC1A.D, IC3A.QS; no longer IC1A.QS, IC2A.D
- net N$68: now also IC3A.Q4; no longer IC1A.Q4
- net N$69: now also IC3A.Q3; no longer IC1A.Q3
- net N$70: now also IC3A.Q5; no longer IC1A.Q5
Other:
- moved on the sheet: IC1

Commit message: Fixing ERC errors
Parts:
- JP1: value (none) -> CON
Connections:
- net +5V: now also JP1.3
Changed lines of the file:
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@@
 <part name="UL2" library="nixie" deviceset="IN-14" device=""/>
 <part name="Q2" library="nixie" deviceset="K155ID1" device=""/>
-<part name="JP1" library="pinhead" deviceset="PINHD-1X8" device=""/>
+<part name="JP1" library="pinhead" deviceset="PINHD-1X8" device="" value="CON"/>
 <part name="Q3" library="nixie" deviceset="K155ID1" device=""/>
 <part name="UL3" library="nixie" deviceset="IN-14" device=""/>
@@
 <part name="P+4" library="supply1" deviceset="+5V" device=""/>
 <part name="P+5" library="supply1" deviceset="+5V" device=""/>
+<part name="VDD1" library="supply1" deviceset="VDD" device=""/>
+<part name="P+1" library="supply1" deviceset="+5V" device=""/>
 </parts>
 <sheets>
@@
 <instance part="P+4" gate="1" x="50.8" y="-38.1"/>
 <instance part="P+5" gate="1" x="50.8" y="-83.82"/>
+<instance part="VDD1" gate="G$1" x="-78.74" y="48.26"/>
+<instance part="P+1" gate="1" x="-71.12" y="48.26"/>
 </instances>
 <busses>
@@
 <wire x1="-40.64" y1="30.48" x2="-27.94" y2="30.48" width="0.1524" layer="91"/>
 <wire x1="-27.94" y1="30.48" x2="-10.16" y2="30.48" width="0.1524" layer="91"/>
-<wire x1="-10.16" y1="-76.2" x2="-27.94" y2="-76.2" width="0.1524" layer="91"/>
 <wire x1="-27.94" y1="-76.2" x2="-27.94" y2="30.48" width="0.1524" layer="91"/>
 <junction x="-27.94" y="30.48"/>
 <pinref part="IC3" gate="A" pin="OE"/>
 <pinref part="IC1" gate="A" pin="OE"/>
+<wire x1="-10.16" y1="-76.2" x2="-27.94" y2="-76.2" width="0.1524" layer="91"/>
 </segment>
 </net>
@@
 <pinref part="P+5" gate="1" pin="+5V"/>
 </segment>
+<segment>
+<pinref part="JP1" gate="A" pin="3"/>
+<pinref part="VDD1" gate="G$1" pin="VDD"/>
+<wire x1="-60.96" y1="38.1" x2="-71.12" y2="38.1" width="0.1524" layer="91"/>
+<wire x1="-71.12" y1="38.1" x2="-78.74" y2="38.1" width="0.1524" layer="91"/>
+<wire x1="-78.74" y1="38.1" x2="-78.74" y2="45.72" width="0.1524" layer="91"/>
+<pinref part="P+1" gate="1" pin="+5V"/>
+<wire x1="-71.12" y1="45.72" x2="-71.12" y2="38.1" width="0.1524" layer="91"/>
+<junction x="-71.12" y="38.1"/>
+</segment>
 </net>
 </nets>
 </sheet>
 </sheets>
+<errors>
+</errors>
 </schematic>
 </drawing>

Commit message: .
Parts:
- R1, R2, R3, R4: value 10K -> 10k; device rcl:R-EU_R1206 -> SparkFun-Passives:RESISTOR1206
Changed lines of the file:
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@@
 <layer number="48" name="Document" color="7" fill="1" visible="no" active="no"/>
 <layer number="49" name="Reference" color="7" fill="1" visible="no" active="no"/>
+<layer number="50" name="dxf" color="7" fill="1" visible="no" active="no"/>
 <layer number="51" name="tDocu" color="7" fill="1" visible="no" active="no"/>
 <layer number="52" name="bDocu" color="7" fill="1" visible="no" active="no"/>
+<layer number="53" name="tGND_GNDA" color="7" fill="9" visible="no" active="no"/>
+<layer number="54" name="bGND_GNDA" color="1" fill="9" visible="no" active="no"/>
+<layer number="56" name="wert" color="7" fill="1" visible="no" active="no"/>
 <layer number="91" name="Nets" color="2" fill="1" visible="yes" active="yes"/>
 <layer number="92" name="Busses" color="1" fill="1" visible="yes" active="yes"/>
@@
 <layer number="97" name="Info" color="7" fill="1" visible="yes" active="yes"/>
 <layer number="98" name="Guide" color="6" fill="1" visible="yes" active="yes"/>
+<layer number="100" name="Muster" color="7" fill="1" visible="no" active="no"/>
+<layer number="101" name="Patch_Top" color="12" fill="4" visible="no" active="yes"/>
+<layer number="102" name="Vscore" color="7" fill="1" visible="no" active="yes"/>
+<layer number="103" name="tMap" color="7" fill="1" visible="no" active="yes"/>
+<layer number="104" name="Name" color="16" fill="1" visible="no" active="yes"/>
+<layer number="105" name="tPlate" color="7" fill="1" visible="no" active="yes"/>
+<layer number="106" name="bPlate" color="7" fill="1" visible="no" active="yes"/>
+<layer number="107" name="Crop" color="7" fill="1" visible="no" active="yes"/>
+<layer number="116" name="Patch_BOT" color="9" fill="4" visible="no" active="yes"/>
+<layer number="121" name="_tsilk" color="7" fill="1" visible="no" active="yes"/>
+<layer number="122" name="_bsilk" color="7" fill="1" visible="no" active="yes"/>
+<layer number="125" name="_tNames" color="7" fill="1" visible="no" active="yes"/>
+<layer number="144" name="Drill_legend" color="7" fill="1" visible="no" active="yes"/>
+<layer number="151" name="HeatSink" color="7" fill="1" visible="no" active="yes"/>
+<layer number="200" name="200bmp" color="1" fill="10" visible="no" active="yes"/>
+<layer number="201" name="201bmp" color="2" fill="10" visible="no" active="yes"/>
+<layer number="202" name="202bmp" color="3" fill="10" visible="no" active="yes"/>
+<layer number="203" name="203bmp" color="4" fill="10" visible="no" active="yes"/>
+<layer number="204" name="204bmp" color="5" fill="10" visible="no" active="yes"/>
+<layer number="205" name="205bmp" color="6" fill="10" visible="no" active="yes"/>
+<layer number="206" name="206bmp" color="7" fill="10" visible="no" active="yes"/>
+<layer number="207" name="207bmp" color="8" fill="10" visible="no" active="yes"/>
+<layer number="208" name="208bmp" color="9" fill="10" visible="no" active="yes"/>
+<layer number="209" name="209bmp" color="7" fill="1" visible="no" active="yes"/>
+<layer number="210" name="210bmp" color="7" fill="1" visible="no" active="yes"/>
+<layer number="211" name="211bmp" color="7" fill="1" visible="no" active="yes"/>
+<layer number="212" name="212bmp" color="7" fill="1" visible="no" active="yes"/>
+<layer number="213" name="213bmp" color="7" fill="1" visible="no" active="yes"/>
+<layer number="214" name="214bmp" color="7" fill="1" visible="no" active="yes"/>
+<layer number="215" name="215bmp" color="7" fill="1" visible="no" active="yes"/>
+<layer number="216" name="216bmp" color="7" fill="1" visible="no" active="yes"/>
+<layer number="217" name="217bmp" color="18" fill="1" visible="no" active="no"/>
+<layer number="218" name="218bmp" color="19" fill="1" visible="no" active="no"/>
+<layer number="219" name="219bmp" color="20" fill="1" visible="no" active="no"/>
+<layer number="220" name="220bmp" color="21" fill="1" visible="no" active="no"/>
+<layer number="221" name="221bmp" color="22" fill="1" visible="no" active="no"/>
+<layer number="222" name="222bmp" color="23" fill="1" visible="no" active="no"/>
+<layer number="223" name="223bmp" color="24" fill="1" visible="no" active="no"/>
+<layer number="224" name="224bmp" color="25" fill="1" visible="no" active="no"/>
+<layer number="250" name="Descript" color="3" fill="1" visible="no" active="no"/>
+<layer number="251" name="SMDround" color="12" fill="11" visible="no" active="no"/>
+<layer number="254" name="cooling" color="7" fill="1" visible="no" active="yes"/>
 </layers>
 <schematic xreflabel="%F%N/%S.%C%R" xrefpart="/%S.%C%R">
@@
 <part name="Q1" library="nixie" deviceset="K155ID1" device=""/>
 <part name="UL1" library="nixie" deviceset="IN-14" device=""/>
-<part name="R1" library="rcl" deviceset="R-EU_" device="R1206" value="10K"/>
-<part name="R2" library="rcl" deviceset="R-EU_" device="R1206" value="10K"/>
 <part name="UL2" library="nixie" deviceset="IN-14" device=""/>
 <part name="Q2" library="nixie" deviceset="K155ID1" device=""/>
@@
 <part name="Q4" library="nixie" deviceset="K155ID1" device=""/>
 <part name="UL4" library="nixie" deviceset="IN-14" device=""/>
-<part name="R3" library="rcl" deviceset="R-EU_" device="R1206" value="10K"/>
-<part name="R4" library="rcl" deviceset="R-EU_" device="R1206" value="10K"/>
 <part name="IC3" library="40xx" deviceset="4094" device="D"/>
 <part name="IC1" library="40xx" deviceset="4094" device="D"/>
@@
 <part name="VDD1" library="supply1" deviceset="VDD" device=""/>
 <part name="P+1" library="supply1" deviceset="+5V" device=""/>
+<part name="R1" library="SparkFun-Passives" deviceset="RESISTOR" device="1206" value="10k"/>
+<part name="R2" library="SparkFun-Passives" deviceset="RESISTOR" device="1206" value="10k"/>
+<part name="R3" library="SparkFun-Passives" deviceset="RESISTOR" device="1206" value="10k"/>
+<part name="R4" library="SparkFun-Passives" deviceset="RESISTOR" device="1206" value="10k"/>
 </parts>
 <sheets>
@@
 <instance part="Q1" gate="G$1" x="73.66" y="40.64"/>
 <instance part="UL1" gate="G$1" x="109.22" y="43.18"/>
-<instance part="R1" gate="G$1" x="104.14" y="76.2"/>
-<instance part="R2" gate="G$1" x="104.14" y="30.48"/>
 <instance part="UL2" gate="G$1" x="109.22" y="-2.54"/>
 <instance part="Q2" gate="G$1" x="73.66" y="-5.08"/>
@@
 <instance part="Q4" gate="G$1" x="73.66" y="-111.76"/>
 <instance part="UL4" gate="G$1" x="109.22" y="-109.22"/>
-<instance part="R3" gate="G$1" x="104.14" y="-30.48"/>
-<instance part="R4" gate="G$1" x="104.14" y="-76.2"/>
 <instance part="IC3" gate="A" x="5.08" y="25.4"/>
 <instance part="IC1" gate="A" x="5.08" y="-81.28"/>
@@
 <instance part="VDD1" gate="G$1" x="-78.74" y="48.26"/>
 <instance part="P+1" gate="1" x="-71.12" y="48.26"/>
+<instance part="R1" gate="G$1" x="104.14" y="76.2"/>
+<instance part="R2" gate="G$1" x="104.14" y="30.48"/>
+<instance part="R3" gate="G$1" x="104.14" y="-30.48"/>
+<instance part="R4" gate="G$1" x="104.14" y="-76.2"/>
 </instances>
 <busses>
@@
 <segment>
 <pinref part="UL1" gate="G$1" pin="A"/>
+<wire x1="99.06" y1="71.12" x2="99.06" y2="76.2" width="0.1524" layer="91"/>
 <pinref part="R1" gate="G$1" pin="1"/>
-<wire x1="99.06" y1="71.12" x2="99.06" y2="76.2" width="0.1524" layer="91"/>
 </segment>
 </net>
 <net name="200V" class="0">
 <segment>
-<pinref part="R1" gate="G$1" pin="2"/>
 <wire x1="109.22" y1="76.2" x2="111.76" y2="76.2" width="0.1524" layer="91"/>
 <label x="111.76" y="76.2" size="1.778" layer="95" xref="yes"/>
-</segment>
-<segment>
-<pinref part="R2" gate="G$1" pin="2"/>
+<pinref part="R1" gate="G$1" pin="2"/>
+</segment>
+<segment>
 <wire x1="109.22" y1="30.48" x2="111.76" y2="30.48" width="0.1524" layer="91"/>
 <label x="111.76" y="30.48" size="1.778" layer="95" xref="yes"/>
+<pinref part="R2" gate="G$1" pin="2"/>
 </segment>
 <segment>
@@
 </segment>
 <segment>
-<pinref part="R3" gate="G$1" pin="2"/>
 <wire x1="109.22" y1="-30.48" x2="111.76" y2="-30.48" width="0.1524" layer="91"/>
 <label x="111.76" y="-30.48" size="1.778" layer="95" xref="yes"/>
-</segment>
-<segment>
-<pinref part="R4" gate="G$1" pin="2"/>
+<pinref part="R3" gate="G$1" pin="2"/>
+</segment>
+<segment>
 <wire x1="109.22" y1="-76.2" x2="111.76" y2="-76.2" width="0.1524" layer="91"/>
 <label x="111.76" y="-76.2" size="1.778" layer="95" xref="yes"/>
+<pinref part="R4" gate="G$1" pin="2"/>
 </segment>
 </net>
@@
 <segment>
 <pinref part="UL2" gate="G$1" pin="A"/>
+<wire x1="99.06" y1="25.4" x2="99.06" y2="30.48" width="0.1524" layer="91"/>
 <pinref part="R2" gate="G$1" pin="1"/>
-<wire x1="99.06" y1="25.4" x2="99.06" y2="30.48" width="0.1524" layer="91"/>
 </segment>
 </net>
@@
 <net name="N$64" class="0">
 <segment>
-<pinref part="R3" gate="G$1" pin="1"/>
 <pinref part="UL3" gate="G$1" pin="A"/>
 <wire x1="99.06" y1="-30.48" x2="99.06" y2="-35.56" width="0.1524" layer="91"/>
+<pinref part="R3" gate="G$1" pin="1"/>
 </segment>
 </net>
@@
 <segment>
 <pinref part="UL4" gate="G$1" pin="A"/>
+<wire x1="99.06" y1="-81.28" x2="99.06" y2="-76.2" width="0.1524" layer="91"/>
 <pinref part="R4" gate="G$1" pin="1"/>
-<wire x1="99.06" y1="-81.28" x2="99.06" y2="-76.2" width="0.1524" layer="91"/>
-</segment>
-</net>
+</segment>
+</net>
