File: controller.sch (EAGLE design)
At the start: 42 parts, among them IC1 MC34063AD, IC2 7805T, IC3 MEGA8-AI, Q1 IRF840, Q2 32768Hz, Q3 4MHz, T1 BC857, U1 DS1307Z

Commit message: Finishing extra components
Parts:
- added C10: 100n, resistor:C-EUC0805K
- added CN1: (no value), adafruit:DCBARRELPTH
- added U$1: RCH110NP, nixie:RCH110NP
- JP3: value EXT -> EXTERNAL; device pinhead:PINHD-1X9/90 -> pinhead:PINHD-1X10/90
Connections:
- net +5V: now also C10.1
- net GND: now also C10.2, CN1.GND, CN1.GNDBREAK, JP3.10, JP3.4; no longer JP3.9
- net N$29: now also CN1.PWR
- net N$33: now also JP3.9; no longer JP3.8
- net N$34: now also JP3.8; no longer JP3.7
- net N$35: now also JP3.7; no longer JP3.6
- net N$36: now also JP3.6; no longer JP3.5
- net N$37: now also JP3.5; no longer JP3.4
- net N$4: now also U$1.2
- net N$7: now also U$1.1
Other:
- moved on the sheet: JP1

Commit message: Update
Parts:
- removed JP1: POWER +12V, pinhead:PINHD-1X2/90
- removed JP3: EXTERNAL, pinhead:PINHD-1X10/90
Connections:
- removed net N$21: IC3.PD0(RXD), JP3.2
- removed net N$22: IC3.PD1(TXD), JP3.3
- removed net N$33: IC3.PD7(AIN1), JP3.9
- removed net N$34: IC3.PD6(AIN0), JP3.8
- removed net N$35: IC3.PD5(T1), JP3.7
- removed net N$36: IC3.PD4(XCK/T0), JP3.6
- removed net N$37: IC3.PD3(INT1), JP3.5
- net +5V: no longer JP3.1
- net GND: no longer JP1.1, JP3.10, JP3.4
- net N$29: no longer JP1.2
Changed lines of the file:
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@@
 <part name="D4" library="adafruit" deviceset="1N4004" device=""/>
 <part name="GND1" library="supply1" deviceset="GND" device=""/>
-<part name="JP1" library="pinhead" deviceset="PINHD-1X2" device="/90" value="POWER +12V"/>
 <part name="JP2" library="pinhead" deviceset="PINHD-1X6" device="/90" value="BUTTONS"/>
 <part name="R7" library="resistor" deviceset="R-EU_" device="M0805" value="10K"/>
@@
 <part name="P+9" library="supply1" deviceset="+5V" device=""/>
 <part name="GND7" library="supply1" deviceset="GND" device=""/>
-<part name="P+8" library="supply1" deviceset="+5V" device=""/>
-<part name="GND6" library="supply1" deviceset="GND" device=""/>
 <part name="BAT1" library="sn2032" deviceset="SN2032" device="" value="3.3V"/>
 <part name="Q2" library="crystal" deviceset="CRYSTAL" device="TC38H" value="32768Hz"/>
@@
 <part name="R15" library="resistor" deviceset="R-EU_" device="M0805" value="1K"/>
 <part name="U$1" library="nixie" deviceset="RCH110NP" device=""/>
-<part name="GND10" library="supply1" deviceset="GND" device=""/>
-<part name="JP3" library="pinhead" deviceset="PINHD-1X10" device="/90" value="EXTERNAL"/>
 <part name="CN1" library="adafruit" deviceset="DCBARREL" device="PTH"/>
 <part name="C10" library="resistor" deviceset="C-EU" device="C0805K" value="100n"/>
@@
 <instance part="D4" gate="1" x="-119.38" y="58.42" rot="R90"/>
 <instance part="GND1" gate="1" x="116.84" y="27.94"/>
-<instance part="JP1" gate="G$1" x="-160.02" y="76.2" rot="R180"/>
 <instance part="JP2" gate="A" x="86.36" y="-43.18"/>
 <instance part="R7" gate="G$1" x="60.96" y="-30.48" rot="R90"/>
@@
 <instance part="P+9" gate="1" x="81.28" y="-167.64"/>
 <instance part="GND7" gate="1" x="81.28" y="-195.58"/>
-<instance part="P+8" gate="1" x="71.12" y="-66.04"/>
-<instance part="GND6" gate="1" x="71.12" y="-106.68"/>
 <instance part="BAT1" gate="1" x="91.44" y="-86.36" rot="R90"/>
 <instance part="Q2" gate="G$1" x="91.44" y="-71.12" rot="R90"/>
@@
 <instance part="R15" gate="G$1" x="17.78" y="-154.94" rot="R180"/>
 <instance part="U$1" gate="G$1" x="76.2" y="73.66"/>
-<instance part="GND10" gate="1" x="71.12" y="-81.28" rot="R270"/>
-<instance part="JP3" gate="A" x="81.28" y="-83.82"/>
 <instance part="CN1" gate="G$1" x="-154.94" y="53.34"/>
 <instance part="C10" gate="G$1" x="162.56" y="-73.66"/>
@@
 <wire x1="-96.52" y1="30.48" x2="-109.22" y2="30.48" width="0.1524" layer="91"/>
 <wire x1="-109.22" y1="30.48" x2="-119.38" y2="30.48" width="0.1524" layer="91"/>
-<wire x1="-119.38" y1="30.48" x2="-142.24" y2="30.48" width="0.1524" layer="91"/>
+<wire x1="-119.38" y1="30.48" x2="-147.32" y2="30.48" width="0.1524" layer="91"/>
 <wire x1="-22.86" y1="30.48" x2="-22.86" y2="33.02" width="0.1524" layer="91"/>
 <pinref part="C2" gate="G$1" pin="2"/>
@@
 <pinref part="GND1" gate="1" pin="GND"/>
 <junction x="116.84" y="30.48"/>
-<pinref part="JP1" gate="G$1" pin="1"/>
-<wire x1="-157.48" y1="73.66" x2="-142.24" y2="73.66" width="0.1524" layer="91"/>
-<wire x1="-142.24" y1="73.66" x2="-142.24" y2="30.48" width="0.1524" layer="91"/>
 <pinref part="CN1" gate="G$1" pin="GND"/>
 <wire x1="-152.4" y1="50.8" x2="-147.32" y2="50.8" width="0.1524" layer="91"/>
 <wire x1="-147.32" y1="50.8" x2="-147.32" y2="30.48" width="0.1524" layer="91"/>
-<wire x1="-147.32" y1="30.48" x2="-142.24" y2="30.48" width="0.1524" layer="91"/>
-<junction x="-142.24" y="30.48"/>
 <pinref part="CN1" gate="G$1" pin="GNDBREAK"/>
 <wire x1="-152.4" y1="53.34" x2="-147.32" y2="53.34" width="0.1524" layer="91"/>
@@
 </segment>
 <segment>
-<pinref part="GND6" gate="1" pin="GND"/>
-<wire x1="71.12" y1="-96.52" x2="71.12" y2="-104.14" width="0.1524" layer="91"/>
-<wire x1="71.12" y1="-96.52" x2="78.74" y2="-96.52" width="0.1524" layer="91"/>
-<pinref part="JP3" gate="A" pin="10"/>
-</segment>
-<segment>
 <pinref part="GND8" gate="1" pin="GND"/>
 <wire x1="-48.26" y1="-66.04" x2="-48.26" y2="-63.5" width="0.1524" layer="91"/>
@@
 <wire x1="12.7" y1="-137.16" x2="12.7" y2="-142.24" width="0.1524" layer="91"/>
 <pinref part="JP5" gate="A" pin="8"/>
-</segment>
-<segment>
-<pinref part="GND10" gate="1" pin="GND"/>
-<wire x1="73.66" y1="-81.28" x2="78.74" y2="-81.28" width="0.1524" layer="91"/>
-<pinref part="JP3" gate="A" pin="4"/>
 </segment>
 <segment>
@@
 </segment>
 <segment>
-<pinref part="P+8" gate="1" pin="+5V"/>
-<wire x1="78.74" y1="-73.66" x2="71.12" y2="-73.66" width="0.1524" layer="91"/>
-<wire x1="71.12" y1="-73.66" x2="71.12" y2="-68.58" width="0.1524" layer="91"/>
-<pinref part="JP3" gate="A" pin="1"/>
-</segment>
-<segment>
 <pinref part="P+10" gate="1" pin="+5V"/>
 <wire x1="20.32" y1="-124.46" x2="12.7" y2="-124.46" width="0.1524" layer="91"/>
@@
 </segment>
 </net>
-<net name="N$21" class="0">
-<segment>
-<pinref part="IC3" gate="G$1" pin="PD0(RXD)"/>
-<wire x1="20.32" y1="-60.96" x2="66.04" y2="-60.96" width="0.1524" layer="91"/>
-<wire x1="66.04" y1="-60.96" x2="66.04" y2="-76.2" width="0.1524" layer="91"/>
-<wire x1="66.04" y1="-76.2" x2="78.74" y2="-76.2" width="0.1524" layer="91"/>
-<pinref part="JP3" gate="A" pin="2"/>
-</segment>
-</net>
-<net name="N$22" class="0">
-<segment>
-<pinref part="IC3" gate="G$1" pin="PD1(TXD)"/>
-<wire x1="20.32" y1="-63.5" x2="63.5" y2="-63.5" width="0.1524" layer="91"/>
-<wire x1="63.5" y1="-63.5" x2="63.5" y2="-78.74" width="0.1524" layer="91"/>
-<wire x1="63.5" y1="-78.74" x2="78.74" y2="-78.74" width="0.1524" layer="91"/>
-<pinref part="JP3" gate="A" pin="3"/>
-</segment>
-</net>
 <net name="N$23" class="0">
 <segment>
@@
 <net name="N$29" class="0">
 <segment>
-<pinref part="JP1" gate="G$1" pin="2"/>
-<wire x1="-157.48" y1="76.2" x2="-147.32" y2="76.2" width="0.1524" layer="91"/>
-<wire x1="-147.32" y1="76.2" x2="-142.24" y2="76.2" width="0.1524" layer="91"/>
-<wire x1="-142.24" y1="76.2" x2="-142.24" y2="83.82" width="0.1524" layer="91"/>
-<pinref part="F1" gate="G$1" pin="1"/>
-<wire x1="-137.16" y1="83.82" x2="-142.24" y2="83.82" width="0.1524" layer="91"/>
 <pinref part="CN1" gate="G$1" pin="PWR"/>
 <wire x1="-152.4" y1="55.88" x2="-147.32" y2="55.88" width="0.1524" layer="91"/>
-<wire x1="-147.32" y1="55.88" x2="-147.32" y2="76.2" width="0.1524" layer="91"/>
-<junction x="-147.32" y="76.2"/>
+<wire x1="-147.32" y1="55.88" x2="-147.32" y2="83.82" width="0.1524" layer="91"/>
+<pinref part="F1" gate="G$1" pin="1"/>
+<wire x1="-147.32" y1="83.82" x2="-137.16" y2="83.82" width="0.1524" layer="91"/>
 </segment>
 </net>
@@
 </segment>
 </net>
-<net name="N$33" class="0">
-<segment>
-<wire x1="38.1" y1="-93.98" x2="38.1" y2="-78.74" width="0.1524" layer="91"/>
-<pinref part="IC3" gate="G$1" pin="PD7(AIN1)"/>
-<wire x1="38.1" y1="-78.74" x2="20.32" y2="-78.74" width="0.1524" layer="91"/>
-<wire x1="78.74" y1="-93.98" x2="38.1" y2="-93.98" width="0.1524" layer="91"/>
-<pinref part="JP3" gate="A" pin="9"/>
-</segment>
-</net>
-<net name="N$34" class="0">
-<segment>
-<pinref part="IC3" gate="G$1" pin="PD6(AIN0)"/>
-<wire x1="20.32" y1="-76.2" x2="40.64" y2="-76.2" width="0.1524" layer="91"/>
-<wire x1="40.64" y1="-76.2" x2="40.64" y2="-91.44" width="0.1524" layer="91"/>
-<wire x1="78.74" y1="-91.44" x2="40.64" y2="-91.44" width="0.1524" layer="91"/>
-<pinref part="JP3" gate="A" pin="8"/>
-</segment>
-</net>
-<net name="N$35" class="0">
-<segment>
-<pinref part="IC3" gate="G$1" pin="PD5(T1)"/>
-<wire x1="20.32" y1="-73.66" x2="43.18" y2="-73.66" width="0.1524" layer="91"/>
-<wire x1="43.18" y1="-73.66" x2="43.18" y2="-88.9" width="0.1524" layer="91"/>
-<wire x1="78.74" y1="-88.9" x2="43.18" y2="-88.9" width="0.1524" layer="91"/>
-<pinref part="JP3" gate="A" pin="7"/>
-</segment>
-</net>
-<net name="N$36" class="0">
-<segment>
-<pinref part="IC3" gate="G$1" pin="PD4(XCK/T0)"/>
-<wire x1="20.32" y1="-71.12" x2="45.72" y2="-71.12" width="0.1524" layer="91"/>
-<wire x1="45.72" y1="-71.12" x2="45.72" y2="-86.36" width="0.1524" layer="91"/>
-<wire x1="78.74" y1="-86.36" x2="45.72" y2="-86.36" width="0.1524" layer="91"/>
-<pinref part="JP3" gate="A" pin="6"/>
-</segment>
-</net>
-<net name="N$37" class="0">
-<segment>
-<pinref part="IC3" gate="G$1" pin="PD3(INT1)"/>
-<wire x1="20.32" y1="-68.58" x2="48.26" y2="-68.58" width="0.1524" layer="91"/>
-<wire x1="48.26" y1="-68.58" x2="48.26" y2="-83.82" width="0.1524" layer="91"/>
-<wire x1="78.74" y1="-83.82" x2="48.26" y2="-83.82" width="0.1524" layer="91"/>
-<pinref part="JP3" gate="A" pin="5"/>
-</segment>
-</net>

Commit message: .
Parts:
- added C11: 100nF, SparkFun-Passives:CAP0805
- C1: value 200p -> 200pF; device resistor:C-EUC0805K -> SparkFun-Passives:CAP0805
- C10, C2, C5, C6: value 100n -> 100nF; device resistor:C-EUC0805K -> SparkFun-Passives:CAP0805
- C8, C9: device rcl:C-EUC0805K -> SparkFun-Passives:CAP0805
- R1: value 1K -> 1k; device resistor:R-EU_M0805 -> SparkFun-Passives:RESISTOR0805-RES
- R10, R11, R12, R13, R14, R4, R7, R8, R9: value 10K -> 10k; device resistor:R-EU_M0805 -> SparkFun-Passives:RESISTOR0805-RES
- R15: value 1K -> 10k; device resistor:R-EU_M0805 -> SparkFun-Passives:RESISTOR0805-RES
- R3, R6: device resistor:R-EU_0617/22 -> SparkFun-Passives:RESISTORPTH-2W
Connections:
- net +5V: now also C6.1; no longer C5.1
- net GND: now also C11.1
- net N$18: now also R15.2; no longer R15.1
- net N$32: now also R15.1; no longer R15.2
- net N$8: now also C5.1; no longer C6.1
- net N$9: now also C11.2
Other:
- moved on the sheet: C5, C6

Commit message: Controller
Parts:
- removed R10, R7, R8, R9: 10k, SparkFun-Passives:RESISTOR0805-RES
- C1: value 200pF -> 1nF
- C3: value 10u 450V -> 10uF 450V
- C4: value 100n 450V -> 100nF 450V; device resistor:C-EU050-035X075 -> SparkFun-Passives:CAPPTH3
- C7: value 470u -> 470uF
- R2: device resistor:R-EU_M0805 -> SparkFun-Passives:RESISTOR0805-RES
Connections:
- net +5V: no longer R10.2, R7.2, R8.2, R9.2
- net N$13: no longer R8.1
- net N$14: no longer R9.1
- net N$15: no longer R10.1
- net N$3: no longer R7.1
Changed lines of the file:
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@@
 <part name="Q1" library="transistor-fet" deviceset="IRF840" device=""/>
 <part name="IC1" library="mc34063" deviceset="MC34063" device="AD"/>
-<part name="R2" library="resistor" deviceset="R-EU_" device="M0805" value="180"/>
 <part name="R5" library="resistor" deviceset="R-TRIMM" device="3339P" value="200K"/>
 <part name="D2" library="diode" deviceset="1N581*" device="" technology="7-B" value="UF4007"/>
-<part name="C3" library="resistor" deviceset="CPOL-EU" device="E5-13" value="10u 450V"/>
-<part name="C4" library="resistor" deviceset="C-EU" device="050-035X075" value="100n 450V"/>
+<part name="C3" library="resistor" deviceset="CPOL-EU" device="E5-13" value="10uF 450V"/>
 <part name="IC2" library="linear" deviceset="78*" device="T" technology="05"/>
-<part name="C7" library="resistor" deviceset="CPOL-EU" device="E5-13" value="470u"/>
+<part name="C7" library="resistor" deviceset="CPOL-EU" device="E5-13" value="470uF"/>
 <part name="IC3" library="atmel" deviceset="MEGA8" device="-AI"/>
 <part name="D4" library="adafruit" deviceset="1N4004" device=""/>
@@
 <part name="CN1" library="adafruit" deviceset="DCBARREL" device="PTH"/>
 <part name="GND11" library="supply1" deviceset="GND" device=""/>
-<part name="R7" library="SparkFun-Passives" deviceset="RESISTOR" device="0805-RES" value="10k"/>
-<part name="R8" library="SparkFun-Passives" deviceset="RESISTOR" device="0805-RES" value="10k"/>
-<part name="R9" library="SparkFun-Passives" deviceset="RESISTOR" device="0805-RES" value="10k"/>
-<part name="R10" library="SparkFun-Passives" deviceset="RESISTOR" device="0805-RES" value="10k"/>
 <part name="R11" library="SparkFun-Passives" deviceset="RESISTOR" device="0805-RES" value="10k"/>
 <part name="R12" library="SparkFun-Passives" deviceset="RESISTOR" device="0805-RES" value="10k"/>
@@
 <part name="C6" library="SparkFun-Passives" deviceset="CAP" device="0805" value="100nF"/>
 <part name="C2" library="SparkFun-Passives" deviceset="CAP" device="0805" value="100nF"/>
-<part name="C1" library="SparkFun-Passives" deviceset="CAP" device="0805" value="200pF"/>
+<part name="C1" library="SparkFun-Passives" deviceset="CAP" device="0805" value="1nF"/>
 <part name="C10" library="SparkFun-Passives" deviceset="CAP" device="0805" value="100nF"/>
 <part name="C8" library="SparkFun-Passives" deviceset="CAP" device="0805" value="22pF"/>
@@
 <part name="R3" library="SparkFun-Passives" deviceset="RESISTOR" device="PTH-2W" value="0.33"/>
 <part name="R6" library="SparkFun-Passives" deviceset="RESISTOR" device="PTH-2W" value="1.2M"/>
+<part name="C4" library="SparkFun-Passives" deviceset="CAP" device="PTH3" value="100nF 450V"/>
+<part name="R2" library="SparkFun-Passives" deviceset="RESISTOR" device="0805-RES" value="180"/>
 </parts>
 <sheets>
@@
 <instance part="Q1" gate="G$1" x="68.58" y="60.96"/>
 <instance part="IC1" gate="G$1" x="-5.08" y="60.96"/>
-<instance part="R2" gate="G$1" x="-22.86" y="71.12" rot="R90"/>
 <instance part="R5" gate="G$1" x="10.16" y="20.32" rot="R270"/>
 <instance part="D2" gate="G$1" x="86.36" y="63.5"/>
 <instance part="C3" gate="G$1" x="99.06" y="45.72"/>
-<instance part="C4" gate="G$1" x="116.84" y="45.72"/>
 <instance part="IC2" gate="A1" x="-96.52" y="53.34"/>
 <instance part="C7" gate="G$1" x="-71.12" y="43.18"/>
@@
 <instance part="JP2" gate="A" x="86.36" y="-43.18"/>
 <instance part="GND2" gate="1" x="78.74" y="-55.88"/>
-<instance part="P+1" gate="1" x="33.02" y="-15.24"/>
+<instance part="P+1" gate="1" x="78.74" y="-20.32"/>
 <instance part="P+2" gate="1" x="-66.04" y="60.96"/>
 <instance part="GND3" gate="1" x="-35.56" y="-68.58" rot="R270"/>
@@
 <instance part="CN1" gate="G$1" x="-154.94" y="53.34"/>
 <instance part="GND11" gate="1" x="162.56" y="-83.82"/>
-<instance part="R7" gate="G$1" x="60.96" y="-30.48" rot="R90"/>
-<instance part="R8" gate="G$1" x="53.34" y="-30.48" rot="R90"/>
-<instance part="R9" gate="G$1" x="45.72" y="-30.48" rot="R90"/>
-<instance part="R10" gate="G$1" x="38.1" y="-30.48" rot="R90"/>
 <instance part="R11" gate="G$1" x="-33.02" y="-20.32" rot="R90"/>
 <instance part="R12" gate="G$1" x="129.54" y="-111.76" rot="R90"/>
@@
 <instance part="R3" gate="G$1" x="-38.1" y="83.82"/>
 <instance part="R6" gate="G$1" x="30.48" y="20.32"/>
+<instance part="C4" gate="G$1" x="116.84" y="43.18"/>
+<instance part="R2" gate="G$1" x="-22.86" y="71.12" rot="R90"/>
 </instances>
 <busses>
@@
 <segment>
 <pinref part="IC1" gate="G$1" pin="DC"/>
-<pinref part="R2" gate="G$1" pin="1"/>
 <wire x1="-20.32" y1="60.96" x2="-22.86" y2="60.96" width="0.1524" layer="91"/>
 <wire x1="-22.86" y1="60.96" x2="-22.86" y2="66.04" width="0.1524" layer="91"/>
+<pinref part="R2" gate="G$1" pin="1"/>
 </segment>
 </net>
 <net name="N$7" class="0">
 <segment>
-<pinref part="R2" gate="G$1" pin="2"/>
 <wire x1="-22.86" y1="76.2" x2="-22.86" y2="83.82" width="0.1524" layer="91"/>
 <wire x1="-22.86" y1="83.82" x2="12.7" y2="83.82" width="0.1524" layer="91"/>
@@
 <wire x1="76.2" y1="83.82" x2="76.2" y2="81.28" width="0.1524" layer="91"/>
 <pinref part="R3" gate="G$1" pin="2"/>
+<pinref part="R2" gate="G$1" pin="2"/>
 </segment>
 </net>
@@
 <segment>
 <pinref part="D2" gate="G$1" pin="C"/>
-<pinref part="C4" gate="G$1" pin="1"/>
 <wire x1="88.9" y1="63.5" x2="99.06" y2="63.5" width="0.1524" layer="91"/>
 <wire x1="99.06" y1="63.5" x2="116.84" y2="63.5" width="0.1524" layer="91"/>
@@
 <junction x="132.08" y="63.5"/>
 <pinref part="R6" gate="G$1" pin="2"/>
+<pinref part="C4" gate="G$1" pin="1"/>
 </segment>
 <segment>
@@
 <junction x="-22.86" y="30.48"/>
 <junction x="-15.24" y="30.48"/>
-<pinref part="C4" gate="G$1" pin="2"/>
 <wire x1="76.2" y1="30.48" x2="99.06" y2="30.48" width="0.1524" layer="91"/>
 <wire x1="99.06" y1="30.48" x2="116.84" y2="30.48" width="0.1524" layer="91"/>
@@
 <pinref part="C2" gate="G$1" pin="2"/>
 <pinref part="C1" gate="G$1" pin="2"/>
+<pinref part="C4" gate="G$1" pin="2"/>
 </segment>
 <segment>
@@
 <pinref part="IC3" gate="G$1" pin="PC0(ADC0)"/>
 <pinref part="JP2" gate="A" pin="2"/>
-<wire x1="20.32" y1="-38.1" x2="60.96" y2="-38.1" width="0.1524" layer="91"/>
-<wire x1="60.96" y1="-38.1" x2="83.82" y2="-38.1" width="0.1524" layer="91"/>
-<wire x1="60.96" y1="-35.56" x2="60.96" y2="-38.1" width="0.1524" layer="91"/>
-<junction x="60.96" y="-38.1"/>
-<pinref part="R7" gate="G$1" pin="1"/>
+<wire x1="20.32" y1="-38.1" x2="83.82" y2="-38.1" width="0.1524" layer="91"/>
 </segment>
 </net>
@@
 <pinref part="IC3" gate="G$1" pin="PC1(ADC1)"/>
 <pinref part="JP2" gate="A" pin="3"/>
-<wire x1="20.32" y1="-40.64" x2="53.34" y2="-40.64" width="0.1524" layer="91"/>
-<wire x1="53.34" y1="-40.64" x2="83.82" y2="-40.64" width="0.1524" layer="91"/>
-<wire x1="53.34" y1="-35.56" x2="53.34" y2="-40.64" width="0.1524" layer="91"/>
-<junction x="53.34" y="-40.64"/>
-<pinref part="R8" gate="G$1" pin="1"/>
+<wire x1="20.32" y1="-40.64" x2="83.82" y2="-40.64" width="0.1524" layer="91"/>
 </segment>
 </net>
@@
 <pinref part="IC3" gate="G$1" pin="PC2(ADC2)"/>
 <pinref part="JP2" gate="A" pin="4"/>
-<wire x1="20.32" y1="-43.18" x2="45.72" y2="-43.18" width="0.1524" layer="91"/>
-<wire x1="45.72" y1="-43.18" x2="83.82" y2="-43.18" width="0.1524" layer="91"/>
-<wire x1="45.72" y1="-35.56" x2="45.72" y2="-43.18" width="0.1524" layer="91"/>
-<junction x="45.72" y="-43.18"/>
-<pinref part="R9" gate="G$1" pin="1"/>
+<wire x1="20.32" y1="-43.18" x2="83.82" y2="-43.18" width="0.1524" layer="91"/>
 </segment>
 </net>
@@
 <pinref part="IC3" gate="G$1" pin="PC3(ADC3)"/>
 <pinref part="JP2" gate="A" pin="5"/>
-<wire x1="20.32" y1="-45.72" x2="38.1" y2="-45.72" width="0.1524" layer="91"/>
-<wire x1="38.1" y1="-45.72" x2="83.82" y2="-45.72" width="0.1524" layer="91"/>
-<wire x1="38.1" y1="-35.56" x2="38.1" y2="-45.72" width="0.1524" layer="91"/>
-<junction x="38.1" y="-45.72"/>
-<pinref part="R10" gate="G$1" pin="1"/>
+<wire x1="20.32" y1="-45.72" x2="83.82" y2="-45.72" width="0.1524" layer="91"/>
 </segment>
 </net>
 <net name="+5V" class="0">
-<segment>
-<wire x1="38.1" y1="-25.4" x2="38.1" y2="-22.86" width="0.1524" layer="91"/>
-<wire x1="38.1" y1="-22.86" x2="45.72" y2="-22.86" width="0.1524" layer="91"/>
-<wire x1="45.72" y1="-22.86" x2="53.34" y2="-22.86" width="0.1524" layer="91"/>
-<wire x1="53.34" y1="-22.86" x2="60.96" y2="-22.86" width="0.1524" layer="91"/>
-<wire x1="60.96" y1="-22.86" x2="78.74" y2="-22.86" width="0.1524" layer="91"/>
-<wire x1="78.74" y1="-22.86" x2="78.74" y2="-35.56" width="0.1524" layer="91"/>
-<pinref part="JP2" gate="A" pin="1"/>
-<wire x1="78.74" y1="-35.56" x2="83.82" y2="-35.56" width="0.1524" layer="91"/>
-<wire x1="60.96" y1="-25.4" x2="60.96" y2="-22.86" width="0.1524" layer="91"/>
-<wire x1="53.34" y1="-25.4" x2="53.34" y2="-22.86" width="0.1524" layer="91"/>
-<wire x1="45.72" y1="-25.4" x2="45.72" y2="-22.86" width="0.1524" layer="91"/>
-<wire x1="38.1" y1="-22.86" x2="33.02" y2="-22.86" width="0.1524" layer="91"/>
-<wire x1="33.02" y1="-22.86" x2="33.02" y2="-17.78" width="0.1524" layer="91"/>
-<junction x="38.1" y="-22.86"/>
-<junction x="45.72" y="-22.86"/>
-<junction x="53.34" y="-22.86"/>
-<junction x="60.96" y="-22.86"/>
-<pinref part="P+1" gate="1" pin="+5V"/>
-<pinref part="R7" gate="G$1" pin="2"/>
-<pinref part="R8" gate="G$1" pin="2"/>
-<pinref part="R9" gate="G$1" pin="2"/>
-<pinref part="R10" gate="G$1" pin="2"/>
-</segment>
 <segment>
 <wire x1="-83.82" y1="45.72" x2="-83.82" y2="53.34" width="0.1524" layer="91"/>
@@
 <pinref part="JP5" gate="A" pin="3"/>
 </segment>
-</net>
+<segment>
+<wire x1="78.74" y1="-22.86" x2="78.74" y2="-35.56" width="0.1524" layer="91"/>
+<pinref part="JP2" gate="A" pin="1"/>
+<wire x1="78.74" y1="-35.56" x2="83.82" y2="-35.56" width="0.1524" layer="91"/>
+<pinref part="P+1" gate="1" pin="+5V"/>
+</segment>
+</net>

Commit message: .
Connections:
- net N$25: now also Q2.1; no longer Q2.2
- net N$26: now also Q2.2; no longer Q2.1
Other:
- moved on the sheet: Q2
Changed lines of the file:
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@@
 <instance part="GND7" gate="1" x="81.28" y="-195.58"/>
 <instance part="BAT1" gate="1" x="91.44" y="-86.36" rot="R90"/>
-<instance part="Q2" gate="G$1" x="91.44" y="-71.12" rot="R90"/>
+<instance part="Q2" gate="G$1" x="91.44" y="-71.12" rot="R270"/>
 <instance part="Q3" gate="G$1" x="-35.56" y="-58.42" rot="R90"/>
 <instance part="GND8" gate="1" x="-48.26" y="-68.58"/>
@@
 <net name="N$25" class="0">
 <segment>
-<pinref part="Q2" gate="G$1" pin="2"/>
-<wire x1="91.44" y1="-68.58" x2="91.44" y2="-66.04" width="0.1524" layer="91"/>
 <wire x1="91.44" y1="-66.04" x2="96.52" y2="-66.04" width="0.1524" layer="91"/>
 <wire x1="96.52" y1="-66.04" x2="96.52" y2="-68.58" width="0.1524" layer="91"/>
 <pinref part="U1" gate="G$1" pin="X1"/>
 <wire x1="96.52" y1="-68.58" x2="101.6" y2="-68.58" width="0.1524" layer="91"/>
+<pinref part="Q2" gate="G$1" pin="1"/>
+<wire x1="91.44" y1="-68.58" x2="91.44" y2="-66.04" width="0.1524" layer="91"/>
 </segment>
 </net>
 <net name="N$26" class="0">
 <segment>
-<pinref part="Q2" gate="G$1" pin="1"/>
-<wire x1="91.44" y1="-73.66" x2="91.44" y2="-76.2" width="0.1524" layer="91"/>
 <wire x1="91.44" y1="-76.2" x2="96.52" y2="-76.2" width="0.1524" layer="91"/>
 <wire x1="96.52" y1="-76.2" x2="96.52" y2="-73.66" width="0.1524" layer="91"/>
 <pinref part="U1" gate="G$1" pin="X2"/>
 <wire x1="96.52" y1="-73.66" x2="101.6" y2="-73.66" width="0.1524" layer="91"/>
-</segment>
-</net>
+<pinref part="Q2" gate="G$1" pin="2"/>
+<wire x1="91.44" y1="-73.66" x2="91.44" y2="-76.2" width="0.1524" layer="91"/>
+</segment>
+</net>
