File: controller.sch (EAGLE design)
At the start: 40 parts, among them IC1 MC34063AD, IC2 7805T, IC3 MEGA8-AI, Q1 IRF840, Q2 32768Hz, Q3 4MHz, T1 BC857, U1 DS1307Z

Commit message: Controller prototype finished
Parts:
- removed C7: 470uF, resistor:CPOL-EUE5-13
- added C12: 100uF, rcl:CPOL-EUE3.5-8
- R5: value 200K -> (none); device resistor:R-TRIMM3339P -> rcl:R-TRIMM64Z
Connections:
- net +5V: now also C12.+; no longer C7.+
- net GND: now also C12.-; no longer C7.-
- net N$10: now also R5.A; no longer R5.E
- net N$11: now also R5.E; no longer R5.A
Changed lines of the file:
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@@
 <part name="Q1" library="transistor-fet" deviceset="IRF840" device=""/>
 <part name="IC1" library="mc34063" deviceset="MC34063" device="AD"/>
-<part name="R5" library="resistor" deviceset="R-TRIMM" device="3339P" value="200K"/>
 <part name="D2" library="diode" deviceset="1N581*" device="" technology="7-B" value="UF4007"/>
 <part name="C3" library="resistor" deviceset="CPOL-EU" device="E5-13" value="10uF 450V"/>
 <part name="IC2" library="linear" deviceset="78*" device="T" technology="05"/>
-<part name="C7" library="resistor" deviceset="CPOL-EU" device="E5-13" value="470uF"/>
 <part name="IC3" library="atmel" deviceset="MEGA8" device="-AI"/>
 <part name="D4" library="adafruit" deviceset="1N4004" device=""/>
@@
 <part name="C4" library="SparkFun-Passives" deviceset="CAP" device="PTH3" value="100nF 450V"/>
 <part name="R2" library="SparkFun-Passives" deviceset="RESISTOR" device="0805-RES" value="180"/>
+<part name="C12" library="rcl" deviceset="CPOL-EU" device="E3.5-8" value="100uF"/>
+<part name="R5" library="rcl" deviceset="R-TRIMM" device="64Z"/>
 </parts>
 <sheets>
@@
 <instance part="Q1" gate="G$1" x="68.58" y="60.96"/>
 <instance part="IC1" gate="G$1" x="-5.08" y="60.96"/>
-<instance part="R5" gate="G$1" x="10.16" y="20.32" rot="R270"/>
 <instance part="D2" gate="G$1" x="86.36" y="63.5"/>
 <instance part="C3" gate="G$1" x="99.06" y="45.72"/>
 <instance part="IC2" gate="A1" x="-96.52" y="53.34"/>
-<instance part="C7" gate="G$1" x="-71.12" y="43.18"/>
 <instance part="IC3" gate="G$1" x="-5.08" y="-63.5"/>
 <instance part="D4" gate="1" x="-119.38" y="58.42" rot="R90"/>
@@
 <instance part="C4" gate="G$1" x="116.84" y="43.18"/>
 <instance part="R2" gate="G$1" x="-22.86" y="71.12" rot="R90"/>
+<instance part="C12" gate="G$1" x="-71.12" y="43.18"/>
+<instance part="R5" gate="G$1" x="10.16" y="20.32" rot="R270"/>
 </instances>
 <busses>
@@
 <wire x1="-15.24" y1="45.72" x2="-5.08" y2="45.72" width="0.1524" layer="91"/>
 <wire x1="-5.08" y1="45.72" x2="-5.08" y2="20.32" width="0.1524" layer="91"/>
-<pinref part="R5" gate="G$1" pin="E"/>
 <wire x1="-5.08" y1="20.32" x2="5.08" y2="20.32" width="0.1524" layer="91"/>
 <junction x="-15.24" y="45.72"/>
 <pinref part="R4" gate="G$1" pin="2"/>
 <pinref part="C2" gate="G$1" pin="1"/>
+<pinref part="R5" gate="G$1" pin="A"/>
 </segment>
 </net>
 <net name="N$11" class="0">
 <segment>
-<pinref part="R5" gate="G$1" pin="A"/>
 <wire x1="15.24" y1="20.32" x2="20.32" y2="20.32" width="0.1524" layer="91"/>
-<pinref part="R5" gate="G$1" pin="S"/>
 <wire x1="20.32" y1="20.32" x2="25.4" y2="20.32" width="0.1524" layer="91"/>
 <wire x1="10.16" y1="15.24" x2="10.16" y2="12.7" width="0.1524" layer="91"/>
@@
 <junction x="20.32" y="20.32"/>
 <pinref part="R6" gate="G$1" pin="1"/>
+<pinref part="R5" gate="G$1" pin="E"/>
+<pinref part="R5" gate="G$1" pin="S"/>
 </segment>
 </net>
@@
 <junction x="-83.82" y="30.48"/>
 <junction x="-109.22" y="30.48"/>
-<pinref part="C7" gate="G$1" pin="-"/>
 <wire x1="-71.12" y1="38.1" x2="-71.12" y2="30.48" width="0.1524" layer="91"/>
 <junction x="-71.12" y="30.48"/>
@@
 <pinref part="C1" gate="G$1" pin="2"/>
 <pinref part="C4" gate="G$1" pin="2"/>
+<pinref part="C12" gate="G$1" pin="-"/>
 </segment>
 <segment>
@@
 <pinref part="IC2" gate="A1" pin="VO"/>
 <wire x1="-83.82" y1="53.34" x2="-86.36" y2="53.34" width="0.1524" layer="91"/>
-<pinref part="C7" gate="G$1" pin="+"/>
 <wire x1="-83.82" y1="53.34" x2="-71.12" y2="53.34" width="0.1524" layer="91"/>
 <wire x1="-71.12" y1="53.34" x2="-71.12" y2="45.72" width="0.1524" layer="91"/>
@@
 <wire x1="-66.04" y1="53.34" x2="-66.04" y2="58.42" width="0.1524" layer="91"/>
 <pinref part="C6" gate="G$1" pin="1"/>
-</segment>
-<segment>
+<pinref part="C12" gate="G$1" pin="+"/>
+</segment>
+<segment>

Commit message: Correct pnp transistor pinout
Parts:
- removed T1: BC857, transistor:-PNP-SOT23-BCE
- added Q6: BC857, SparkFun-DiscreteSemi:TRANSISTOR_PNPSMD
Connections:
- net GND: now also Q6.C; no longer T1.C
- net N$1: now also Q6.E; no longer T1.E
- net N$2: now also Q6.B; no longer T1.B
Changed lines of the file:
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@@
 <setting verticaltext="up"/>
 </settings>
-<grid distance="0.1" unitdist="inch" unit="inch" style="lines" multiple="1" display="no" altdistance="0.01" altunitdist="inch" altunit="inch"/>
+<grid distance="0.1" unitdist="inch" unit="inch" style="dots" multiple="1" display="yes" altdistance="0.01" altunitdist="inch" altunit="inch"/>
 <layers>
 <layer number="1" name="Top" color="4" fill="1" visible="no" active="no"/>
@@
 </classes>
 <parts>
-<part name="T1" library="transistor" deviceset="*-PNP-" device="SOT23-BCE" value="BC857"/>
 <part name="D1" library="diode" deviceset="1N4148" device="DO35-7"/>
 <part name="Q1" library="transistor-fet" deviceset="IRF840" device=""/>
@@
 <part name="C12" library="rcl" deviceset="CPOL-EU" device="E3.5-8" value="100uF"/>
 <part name="R5" library="rcl" deviceset="R-TRIMM" device="64Z"/>
+<part name="Q6" library="SparkFun-DiscreteSemi" deviceset="TRANSISTOR_PNP" device="SMD" value="BC857"/>
 </parts>
 <sheets>
@@
 </plain>
 <instances>
-<instance part="T1" gate="G$1" x="45.72" y="45.72"/>
 <instance part="D1" gate="G$1" x="43.18" y="58.42"/>
 <instance part="Q1" gate="G$1" x="68.58" y="60.96"/>
@@
 <instance part="C12" gate="G$1" x="-71.12" y="43.18"/>
 <instance part="R5" gate="G$1" x="10.16" y="20.32" rot="R270"/>
+<instance part="Q6" gate="G$1" x="45.72" y="45.72"/>
 </instances>
 <busses>
@@
 <pinref part="D1" gate="G$1" pin="C"/>
 <wire x1="45.72" y1="58.42" x2="48.26" y2="58.42" width="0.1524" layer="91"/>
-<pinref part="T1" gate="G$1" pin="E"/>
 <wire x1="48.26" y1="58.42" x2="48.26" y2="50.8" width="0.1524" layer="91"/>
 <pinref part="Q1" gate="G$1" pin="G"/>
 <wire x1="48.26" y1="58.42" x2="63.5" y2="58.42" width="0.1524" layer="91"/>
 <junction x="48.26" y="58.42"/>
+<pinref part="Q6" gate="G$1" pin="E"/>
 </segment>
 </net>
@@
 <wire x1="40.64" y1="58.42" x2="38.1" y2="58.42" width="0.1524" layer="91"/>
 <wire x1="38.1" y1="58.42" x2="38.1" y2="45.72" width="0.1524" layer="91"/>
-<pinref part="T1" gate="G$1" pin="B"/>
 <wire x1="38.1" y1="45.72" x2="43.18" y2="45.72" width="0.1524" layer="91"/>
 <wire x1="38.1" y1="43.18" x2="38.1" y2="45.72" width="0.1524" layer="91"/>
@@
 <junction x="38.1" y="58.42"/>
 <pinref part="R1" gate="G$1" pin="2"/>
+<pinref part="Q6" gate="G$1" pin="B"/>
 </segment>
 </net>
@@
 <segment>
 <wire x1="38.1" y1="33.02" x2="38.1" y2="30.48" width="0.1524" layer="91"/>
-<pinref part="T1" gate="G$1" pin="C"/>
 <wire x1="38.1" y1="30.48" x2="48.26" y2="30.48" width="0.1524" layer="91"/>
 <wire x1="48.26" y1="30.48" x2="48.26" y2="40.64" width="0.1524" layer="91"/>
@@
 <pinref part="C4" gate="G$1" pin="2"/>
 <pinref part="C12" gate="G$1" pin="-"/>
-</segment>
-<segment>
+<pinref part="Q6" gate="G$1" pin="C"/>
+</segment>
+<segment>
